File: DCDC_converter/DCDC_converter.kicad_sch (KiCad schematic)
At the start: 31 parts, among them J1 Conn_01x02_Pin, J2 Conn_01x02_Pin, J3 Conn_01x02_Pin, J4 Conn_01x02_Pin, U1 MP2491C

Commit message: Final version of DC/DC module
Parts:
- added J5: Conn_01x03_Pin, Connector_PinHeader_2.54mm:PinHeader_1x03_P2.54mm_Vertical, symbol Connector:Conn_01x03_Pin
- added J6: Conn_01x02_Pin, Connector_PinHeader_2.54mm:PinHeader_1x02_P2.54mm_Vertical, symbol Connector:Conn_01x02_Pin
Connections:
- net +5V: now also J5.2 (Pin_2); no longer J3.1 (Pin_1), J3.2 (Pin_2)
- new net: J3.1 (Pin_1), J3.2 (Pin_2), J5.1 (Pin_1)
- new net: J5.3 (Pin_3), J6.1 (Pin_1), J6.2 (Pin_2)
Other:
- moved on the sheet: J3
