File: USART.kicad_sch (KiCad schematic)
At the start: 0 parts

Commit message: Added inputs and outputs to the schematic
Parts:
- added U6: FT2232HQ, Package_DFN_QFN:QFN-64-1EP_9x9mm_P0.5mm_EP4.35x4.35mm, symbol Interface_USB:FT2232HQ
Changed lines of the file:
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@@
 	(generator_version "8.0")
 	(paper "A4")
+	(symbol
+		(lib_id "Interface_USB:FT2232HQ")
+		(at 78.74 81.28 0)
+		(unit 1)
+		(exclude_from_sim no)
+		(in_bom yes)
+		(on_board yes)
+		(dnp no)
+		(fields_autoplaced yes)
+		(property "Reference" "U6"
+			(at 93.6341 24.13 0)
+			(effects
+				(font
+					(size 1.27 1.27)
+				)
+				(justify left)
+			)
+		)
+		(property "Value" "FT2232HQ"
+			(at 93.6341 26.67 0)
+			(effects
+				(font
+					(size 1.27 1.27)
+				)
+				(justify left)
+			)
+		)
+		(property "Footprint" "Package_DFN_QFN:QFN-64-1EP_9x9mm_P0.5mm_EP4.35x4.35mm"
+			(at 78.74 81.28 0)
+			(effects
+				(font
+					(size 1.27 1.27)
+				)
+				(hide yes)
+			)
+		)
+		(property "Datasheet" "https://www.ftdichip.com/Support/Documents/DataSheets/ICs/DS_FT2232H.pdf"
+			(at 78.74 81.28 0)
+			(effects
+				(font
+					(size 1.27 1.27)
+				)
+				(hide yes)
+			)
+		)
+		(property "Description" "Hi Speed Double Channel USB UART/FIFO, QFN-64"
+			(at 78.74 81.28 0)
+			(effects
+				(font
+					(size 1.27 1.27)
+				)
+				(hide yes)
+			)
+		)
+		(pin "42"
+		)
+		(pin "48"
+		)
+		(pin "28"
+		)
+		(pin "5"
+		)
+		(pin "53"
+		)
+		(pin "52"
+		)
+		(pin "55"
+		)
+		(pin "57"
+		)
+		(pin "60"
+		)
+		(pin "61"
+		)
+		(pin "3"
+		)
+		(pin "15"
+		)
+		(pin "23"
+		)
+		(pin "35"
+		)
+		(pin "45"
+		)
+		(pin "11"
+		)
+		(pin "65"
+		)
+		(pin "13"
+		)
+		(pin "30"
+		)
+		(pin "36"
+		)
+		(pin "38"
+		)
+		(pin "51"
+		)
+		(pin "59"
+		)
+		(pin "40"
+		)
+		(pin "6"
+		)
+		(pin "20"
+		)
+		(pin "7"
+		)
+		(pin "56"
+		)
+		(pin "37"
+		)
+		(pin "34"
+		)
+		(pin "46"
+		)
+		(pin "16"
+		)
+		(pin "29"
+		)
+		(pin "14"
+		)
+		(pin "2"
+		)
+		(pin "21"
+		)
+		(pin "63"
+		)
+		(pin "41"
+		)
+		(pin "22"
+		)
+		(pin "24"
+		)
+		(pin "27"
+		)
+		(pin "43"
+		)
+		(pin "49"
+		)
+		(pin "54"
+		)
+		(pin "26"
+		)
+		(pin "33"
+		)
+		(pin "12"
+		)
+		(pin "44"
+		)
+		(pin "1"
+		)
+		(pin "17"
+		)
+		(pin "50"
+		)
+		(pin "58"
+		)
+		(pin "39"
+		)
+		(pin "10"
+		)
+		(pin "47"
+		)
+		(pin "4"
+		)
+		(pin "64"
+		)
+		(pin "32"
+		)
+		(pin "8"
+		)
+		(pin "62"
+		)
+		(pin "25"
+		)
+		(pin "18"
+		)
+		(pin "19"
+		)
+		(pin "31"
+		)
+		(pin "9"
+		)
+		(instances
+			(project "LPV01_SHIELD"
+				(path "/235a657c-2000-4f74-9092-d8e0f0a5ea32/bd9cb392-e7f9-4c99-9924-5e1544e553e5"
+					(reference "U6")
+					(unit 1)
+				)
+			)
+		)
+	)
 )
