File: USB_hub.kicad_sch (KiCad schematic)
At the start: 0 parts

Commit message: Added inputs and outputs to the schematic
Parts:
- added J12, J13, J4: USB1035-GF-P-0-B-B, SamacSys_Parts:USB1035GFP0BB, symbol SamacSys_Parts:USB1035-GF-P-0-B-B
- added J14: A-USBSA, SamacSys_Parts:A-USBSA, symbol SamacSys_Parts:A-USBSA
- added J18, J19, J20, J21: Screw_Terminal_01x02, TerminalBlock_Phoenix:TerminalBlock_Phoenix_MKDS-1,5-2_1x02_P5.00mm_Horizontal, symbol Connector:Screw_Terminal_01x02
- added U4: USB2517I-JZX, Package_DFN_QFN:QFN-64-1EP_9x9mm_P0.5mm_EP5.45x5.45mm_ThermalVias, symbol SamacSys_Parts:USB2517I-JZX
- added U7: M24C02-FMN, Package_SO:SOIC-8_3.9x4.9mm_P1.27mm, symbol Memory_EEPROM:M24C02-FMN
Connections:
- new net D1+: J4.A3
- new net D1-: J4.A2
- new net D2+: J4.B3
- new net D2-: J4.B2
- new net GND: J4.A4, J4.B4
- new net VBUS1: J4.A1
- new net VBUS2: J4.B1

Commit message: PCB rebuilt
Changed lines of the file:
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@@
-	)
-	(symbol
-		(lib_id "power:+5V")
-		(at 242.57 52.07 0)
-		(unit 1)
-		(exclude_from_sim no)
-		(in_bom yes)
-		(on_board yes)
-		(dnp no)
-		(fields_autoplaced yes)
-		(property "Reference" "#PWR046"
-			(at 242.57 55.88 0)
-			(effects
-				(font
-					(size 1.27 1.27)
-				)
-				(hide yes)
-			)
-		)
-		(property "Value" "+5V"
-			(at 242.57 46.99 0)
-			(effects
-				(font
-					(size 1.27 1.27)
-				)
-			)
-		)
-		(property "Footprint" ""
-			(at 242.57 52.07 0)
-			(effects
-				(font
-					(size 1.27 1.27)
-				)
-				(hide yes)
-			)
-		)
-		(property "Datasheet" ""
-			(at 242.57 52.07 0)
-			(effects
-				(font
-					(size 1.27 1.27)
-				)
-				(hide yes)
-			)
-		)
-		(property "Description" "Power symbol creates a global label with name \"+5V\""
-			(at 242.57 52.07 0)
-			(effects
-				(font
-					(size 1.27 1.27)
-				)
-				(hide yes)
-			)
-		)
-		(pin "1"
-		)
-		(instances
-			(project "LPV01_SHIELD"
-				(path "/235a657c-2000-4f74-9092-d8e0f0a5ea32/d4abdc1d-30ec-42d0-9d29-446571cc57b4"
-					(reference "#PWR046")
-					(unit 1)
-				)
-			)
-		)
 	)
 	(symbol
